Commit message: Update four_wheel_bot.xacro

File: src/four_wheel_bot/urdf/four_wheel_bot.xacro (robot description, xacro)
@@ -14,4 +14,7 @@
         <box size="${body_length} ${body_width} ${body_height}"/>
       </geometry>
+      <material name="red">
+        <color rgba="1 0 0 1"/>
+      </material>
     </visual>
     <collision>
@@ -36,5 +39,7 @@
           <cylinder radius="${wheel_radius}" length="${wheel_width}"/>
         </geometry>
-        <material name="Gazebo/Black"/>
+        <material name="black">
+          <color rgba="0 0 0 1"/>
+        </material>
       </visual>
       <collision>
@@ -81,5 +86,5 @@
     <material>Gazebo/Yellow</material>
   </gazebo>
-  <!-- === LIDAR Sensor === -->
+  <!-- === LIDAR Sensor (Corrected Plugin) === -->
   <link name="lidar_link">
     <visual>
@@ -110,4 +115,5 @@
   <gazebo reference="lidar_link">
     <sensor name="lidar" type="ray">
+      <pose>0 0 0 0 0 0</pose>
       <update_rate>10</update_rate>
       <visualize>true</visualize>
@@ -126,7 +132,10 @@
         </range>
       </ray>
-      <plugin name="gazebo_ros_laser" filename="libgazebo_ros_laser.so">
-        <topicName>scan</topicName>
-        <frameName>lidar_link</frameName>
+      <plugin name="gazebo_ros_laser_controller" filename="libgazebo_ros_ray_sensor.so">
+        <ros>
+          <remapping>~/out:=scan</remapping>
+        </ros>
+        <update_rate>10.0</update_rate>
+        <frame_name>lidar_link</frame_name>
       </plugin>
     </sensor>
@@ -186,6 +195,6 @@
   <gazebo>
     <plugin name="diff_drive_controller" filename="libgazebo_ros_diff_drive.so">
-      <left_wheel_joint>joint_rl</left_wheel_joint>
-      <right_wheel_joint>joint_rr</right_wheel_joint>
+      <left_joint>joint_rl</left_joint>
+      <right_joint>joint_rr</right_joint>
       <wheel_separation>${body_width}</wheel_separation>
       <wheel_diameter>${2 * wheel_radius}</wheel_diameter>
